File: eagle/projects/shift_register_board/shift_reg.sch (EAGLE design)
At the start: 34 parts, among them U1 SN74HC595N, U2 SN74HC595N, U3 SN74HC595N, U4 SN74HC595N

Commit message: Started board layout
Parts:
- J1: device SparkFun-Connectors:CONN_063.5MM-6 -> shift_register:CONN_06
- J2, J3: device SparkFun-Connectors:CONN_10" -> shift_register:CONN_101X10_WIDE
- J4: device SparkFun-Connectors:CONN_09 -> shift_register:CONN_101X10_WIDE
- R1, R10, R11, R12, R13, R14, R15, R16, R17, R18, R19, R2, R20, R21, R22, R23, R24, R25, R26, R3, R4, R5, R6, R7, R8, R9: device SparkFun-Resistors:RESISTORAXIAL-0.3 -> SparkFun-Resistors:RESISTOR0805
- U1, U2, U3, U4: value SN74HC595N -> SN74HC595D; device SparkFun-IC-Logic:74HC595N -> SparkFun-IC-Logic:74HC595D
Connections:
- net GND: now also J4.10; no longer J4.9
- net I: now also J2.9; no longer J3.9
- net J: now also J2.8; no longer J3.8
- net K: now also J2.7; no longer J3.7
- net L: now also J2.6; no longer J3.6
- net M: now also J2.5; no longer J3.5
- net N: now also J2.4; no longer J3.4
- net O: now also J2.3; no longer J3.3
- net P: now also J2.2; no longer J3.2
- net Q: now also J2.1; no longer J3.1
- net R: now also J3.9; no longer J2.9
- net S: now also J3.8; no longer J2.8
- net T: now also J3.7; no longer J2.7
- net U: now also J3.6; no longer J2.6
- net V: now also J3.5; no longer J2.5
- net W: now also J3.4; no longer J2.4
- net X: now also J3.3; no longer J2.3
- net Y: now also J3.2; no longer J2.2
- net Z: now also J3.1; no longer J2.1
Other:
- moved on the sheet: J1, J2, J3

Commit message: Laid out board with through holes. Ready for pour
Parts:
- removed J1: (no value), shift_register:CONN_06
- added J5: (no value), SparkFun-Connectors:CONN_06LOCK
- J2, J3, J4: device shift_register:CONN_101X10_WIDE -> shift_register:CONN_10"
- R1, R10, R11, R12, R13, R14, R15, R16, R17, R18, R19, R2, R20, R21, R22, R23, R24, R25, R26, R3, R4, R5, R6, R7, R8, R9: device SparkFun-Resistors:RESISTOR0805 -> SparkFun-Resistors:RESISTORAXIAL-0.3
- U1, U2, U3, U4: value SN74HC595D -> SN74HC595N; device SparkFun-IC-Logic:74HC595D -> SparkFun-IC-Logic:74HC595N
Connections:
- net CLOCK: now also J5.5; no longer J1.5
- net DATA: now also J5.3; no longer J1.3
- net GND: now also J5.1; no longer J1.1
- net LATCH: now also J5.4; no longer J1.4
- net OE: now also J5.2; no longer J1.2
- net VCC: now also J5.6; no longer J1.6
Other:
- moved on the sheet: J2, J3, J4
