File: eagle/projects/shift_register_board/shift_reg.brd (EAGLE design)
At the start: 90.9 x 76.2 mm, 34 parts, among them U1 SN74HC595N, U2 SN74HC595N, U3 SN74HC595N, U4 SN74HC595N

Commit message: Added pours and silkscreen text. Ready for images
Routing:
- added copper zone on layer 16, net GND
Other:
- board size 90.9 x 76.2 mm -> 90 x 80 mm
- board text added: "A"
- board text added: "B"
- board text added: "C"
- board text added: "CLOCK"
- board text added: "D"
- board text added: "DATA"
- board text added: "E"
- board text added: "F"
- board text added: "G"
- board text added: "GND"
- board text added: "H"
- board text added: "I"
- board text added: "J"
- board text added: "K"
- board text added: "L"
- board text added: "LATCH"
- board text added: "M"
- board text added: "N"
- board text added: "O"
- board text added: "OE"
- board text added: "P"
- board text added: "Q"
- board text added: "R"
- board text added: "S"
- board text added: "T"
- board text added: "U"
- board text added: "V"
- board text added: "VCC"
- board text added: "W"
- board text added: "X"
- board text added: "Y"
- board text added: "Z"
Changed lines of the file:
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@@
 <setting verticaltext="up"/>
 </settings>
-<grid distance="10" unitdist="mil" unit="mil" style="lines" multiple="1" display="yes" altdistance="5" altunitdist="mil" altunit="mil"/>
+<grid distance="20" unitdist="mil" unit="mil" style="lines" multiple="1" display="yes" altdistance="5" altunitdist="mil" altunit="mil"/>
 <layers>
 <layer number="1" name="Top" color="4" fill="1" visible="yes" active="yes"/>
@@
 <board>
 <plain>
-<wire x1="0" y1="76.19" x2="0" y2="0" width="0.508" layer="20"/>
-<wire x1="0" y1="76.2" x2="90.932" y2="76.2" width="0.508" layer="20"/>
-<wire x1="90.932" y1="76.2" x2="90.932" y2="0" width="0.508" layer="20"/>
-<wire x1="90.932" y1="0" x2="0" y2="0" width="0.508" layer="20"/>
+<wire x1="0" y1="80" x2="0" y2="0" width="0.508" layer="20"/>
+<wire x1="0" y1="0" x2="90" y2="0" width="0.508" layer="20"/>
+<wire x1="90" y1="0" x2="90" y2="80" width="0.508" layer="20"/>
+<wire x1="90" y1="80" x2="0" y2="80" width="0.508" layer="20"/>
+<text x="75.184" y="1.524" size="0.4064" layer="21">GND</text>
+<text x="73.152" y="1.524" size="0.4064" layer="21">OE</text>
+<text x="70.612" y="1.524" size="0.4064" layer="21">DATA</text>
+<text x="67.564" y="1.524" size="0.4064" layer="21">LATCH</text>
+<text x="65.024" y="1.524" size="0.4064" layer="21">CLOCK</text>
+<text x="62.992" y="1.524" size="0.4064" layer="21">VCC</text>
+<text x="2.032" y="41.656" size="1.016" layer="21">Z</text>
+<text x="2.032" y="38.608" size="1.016" layer="21">Y</text>
+<text x="2.032" y="36.068" size="1.016" layer="21">X</text>
+<text x="2.032" y="33.528" size="1.016" layer="21">W</text>
+<text x="2.032" y="30.988" size="1.016" layer="21">V</text>
+<text x="2.032" y="28.448" size="1.016" layer="21">U</text>
+<text x="2.032" y="25.908" size="1.016" layer="21">T</text>
+<text x="2.032" y="23.368" size="1.016" layer="21">S</text>
+<text x="2.032" y="20.828" size="1.016" layer="21">R</text>
+<text x="2.032" y="70.612" size="1.016" layer="21">Q</text>
+<text x="2.032" y="68.072" size="1.016" layer="21">P</text>
+<text x="2.032" y="65.532" size="1.016" layer="21">O</text>
+<text x="2.032" y="62.992" size="1.016" layer="21">N</text>
+<text x="2.032" y="60.452" size="1.016" layer="21">M</text>
+<text x="2.032" y="57.912" size="1.016" layer="21">L</text>
+<text x="2.032" y="55.372" size="1.016" layer="21">K</text>
+<text x="2.032" y="52.832" size="1.016" layer="21">J</text>
+<text x="2.032" y="50.292" size="1.016" layer="21">I</text>
+<text x="57.912" y="74.676" size="1.016" layer="21">A</text>
+<text x="60.452" y="74.676" size="1.016" layer="21">B</text>
+<text x="62.992" y="74.676" size="1.016" layer="21">C</text>
+<text x="65.532" y="74.676" size="1.016" layer="21">D</text>
+<text x="68.072" y="74.676" size="1.016" layer="21">E</text>
+<text x="70.612" y="74.676" size="1.016" layer="21">F</text>
+<text x="73.152" y="74.676" size="1.016" layer="21">G</text>
+<text x="75.692" y="74.676" size="1.016" layer="21">H</text>
 </plain>
 <attributes>
@@
 <contactref element="J4" pad="10"/>
 <polygon width="0.508" layer="1">
-<vertex x="90.932" y="76.2"/>
-<vertex x="73.914" y="76.2"/>
-<vertex x="0" y="76.2"/>
+<vertex x="0" y="0"/>
+<vertex x="0" y="80.01"/>
+<vertex x="22.86" y="80.01"/>
+<vertex x="90.17" y="80.01"/>
+<vertex x="90.17" y="0"/>
 </polygon>
-<wire x1="34.29" y1="53.34" x2="53.34" y2="72.39" width="0" layer="19" extent="1-1"/>
-<wire x1="60.96" y1="44.45" x2="34.29" y2="53.34" width="0" layer="19" extent="1-1"/>
-<wire x1="60.96" y1="24.13" x2="60.96" y2="44.45" width="0" layer="19" extent="1-1"/>
-<wire x1="76.2" y1="4.572" x2="60.96" y2="24.13" width="0" layer="19" extent="1-1"/>
-<wire x1="35.56" y1="21.59" x2="60.96" y2="24.13" width="0" layer="19" extent="1-1"/>
-<wire x1="5.08" y1="48.26" x2="34.29" y2="53.34" width="0" layer="19" extent="1-1"/>
-<wire x1="5.08" y1="19.05" x2="5.08" y2="48.26" width="0" layer="19" extent="1-1"/>
+<polygon width="0.508" layer="16">
+<vertex x="0" y="0"/>
+<vertex x="0" y="80.01"/>
+<vertex x="86.36" y="80.01"/>
+<vertex x="90.17" y="80.01"/>
+<vertex x="90.17" y="2.54"/>
+<vertex x="90.17" y="0"/>
+</polygon>
 </signal>
 <signal name="LATCH">
